File: 2HPico DSP KiCad Design Files/Pico 2HP_Audio/Pico 2HP_Audio.kicad_sch (KiCad schematic)
At the start: 58 parts, among them J1 Conn_01x04_Pin, J2 Conn_01x04_Pin, J3 Conn_01x04_Pin, J4 Conn_01x05_Pin, U1 74LVC1G3157, U2 74LVC1G3157, U3 AMS1117-5.0, U4 LM4040DBZ-10, U5 TL072, U6 PCM5102A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

Commit message: Updated 2HPico DSP schematic, BOM and JLCPCB assy files
BOM changes as a result of further testing: R1 -> 47 ohms, R10,R17->10k.
Parts:
- R1: value 100R -> 47R
Changed lines of the file:
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@@
 			)
 		)
-		(property "Value" "100R"
+		(property "Value" "47R"
 			(at 60.96 147.32 90)
 			(effects
