File: 4HPico DSP KiCad design files/4HPicoDSP.kicad_pcb (KiCad board)
At the start: 2 copper layers, 20.3 x 110 mm, 71 parts, among them J1 PJ3001F, J2 PJ3001F, J3 PJ3001F, J4 PJ3001F, J5 PJ3001F, J6 PJ3001F, J7 Conn_02x05_Odd_Even, J8 Conn_01x04_Pin, SW1 RotaryEncoder_Switch, U3 AMS1117-5.0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

Commit message: Updated to V1.1
Connected middle and bottom GND planes. Added panel .stl file for 3D printing.
Routing:
- net GND: track 254.0 -> 269.6 mm, vias 31 -> 32
Other:
- board text added: "4HPico DSP by Rich Heslip V1.1 5/6/2026"
- board text removed: "4HPico by Rich Heslip V1.0 4/12/2026"
